File: src/RT4K_donut_dongle.kicad_pcb (KiCad board)
At the start: 2 copper layers, 42.2 x 68.1 mm, 48 parts, among them J1 2.54mm Pitch Single Row Femal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, J10 PJ-320, J11 PJ-320, J2 2.54mm Pitch Single Row Femal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, J3 2x5 Pin Double Row 2.54mm Pit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, J4 PJ-320, J5 2x4 Pin Double Row 2.54mm Pit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, J6 2x5 Pin Double Row 2.54mm Pit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, J8 2x4 Pin Double Row 2.54mm Pit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, J9 PJ-320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

Commit message: RC2 updated KiCad files
Parts:
- added R10: 10K OHM 1% 1/8W 0805, Resistor_SMD:R_0805_2012Metric_Pad1.20x1.40mm_HandSolder, B.Cu at (111.4, 96.0)
- moved C5 1.16 mm to (116.8, 95.0)
- moved R21 1.14 mm to (113.4, 96.0), turned to 180 degrees
- renumbered J2 to J1, R10 to R21
Connections:
- net /D13/SCK renamed /D13/SCK (LED)
- R21 pad 1: Net-(U2-1Y) -> +5V
- R21 pad 2: +5V -> Net-(U2-1Y)
Routing:
- net +3V3: track 0.00 -> 7.40 mm
- net +5V: track 66.6 -> 64.9 mm
- net Net-(U2-1Y): track 6.29 -> 7.69 mm
- net /D1/TX: track 43.0 -> 42.1 mm
- net /*D10/SS gsw2 override: vias 0 -> 2
Other:
- board text added: "3v3"
- board text added: "5v"
- board text added: "PU"
