File: src/RT4K_donut_dongle.kicad_sch (KiCad schematic)
At the start: 47 parts, among them J1 2.54mm Pitch Single Row Femal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, J10 PJ-320, J11 PJ-320, J2 2.54mm Pitch Single Row Femal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, J3 2x5 Pin Double Row 2.54mm Pit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, J4 PJ-320, J5 2x4 Pin Double Row 2.54mm Pit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, J6 2x5 Pin Double Row 2.54mm Pit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, J8 2x4 Pin Double Row 2.54mm Pit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, J9 PJ-320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

Commit message: RC2 updated KiCad files
Parts:
- added R10: 10K OHM 1% 1/8W 0805, Resistor_SMD:R_0805_2012Metric_Pad1.20x1.40mm_HandSolder, symbol Library:R_Small
- R21: renamed from R10; now not fitted; now left out of the parts list
Connections:
- net +3V3: now also R10.1
- net +5V: now also R21.1; no longer R21.2
- net at PH1.T, U2.6 (1Y): now also R21.2, R10.2; no longer R21.1

Commit message: updated RC2 info
Parts:
- R21: now fitted
Other:
- note added: "option of 3v3 or 5v for TX pullup"
Changed lines of the file:
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@@
 		)
 	)
+	(text "option of 3v3 or 5v for TX pullup"
+		(exclude_from_sim no)
+		(at 54.61 109.22 0)
+		(effects
+			(font
+				(size 1.27 1.27)
+			)
+		)
+	)
 	(text "L"
 		(exclude_from_sim no)
@@
 		(dnp no)
 		(property "Reference" "R10"
-			(at 53.34 101.6 90)
+			(at 53.34 104.14 90)
 			(effects
 				(font
@@
 		(in_bom no)
 		(on_board yes)
-		(dnp yes)
+		(dnp no)
 		(property "Reference" "R21"
 			(at 53.34 109.22 90)
